File: tinkertechLED.brd (EAGLE design)
At the start: 38.1 x 38.1 mm, 4 parts

Commit message: Final chances before initial production
Parts:
- R1: value (none) -> 100; device SparkFun-Passives:AXIAL-0.3 -> SparkFun-Passives:AXIAL-0.3-KIT
- moved R1 0.25 mm to (19.1, 4.06), turned to 0 degrees
- moved S1 0.25 mm to (19.1, 32.5)
Routing:
- net N$3: track 46.0 -> 31.3 mm, vias 1 -> 0
- net L2: track 38.9 -> 26.5 mm
- net L1: track 34.9 -> 24.1 mm
- net L6: track 18.8 -> 11.3 mm
- net T2: track 28.8 -> 24.7 mm
- net L5: track 21.9 -> 18.2 mm
- net N$2: track 16.3 -> 19.1 mm
- net T3: track 28.4 -> 25.6 mm
- net N$4: track 7.53 -> 4.94 mm, vias 1 -> 0
- net T4: track 37.4 -> 38.4 mm
- net L4: track 27.7 -> 27.1 mm
Other:
- board text added: "+"
- board text added: "www.tinkertech.io Ypsilanti, MI"
