File: tinkertechLED.sch (EAGLE design)
At the start: 4 parts

Commit message: Final chances before initial production
Parts:
- R1: value (none) -> 100; device SparkFun-Passives:RESISTORAXIAL-0.3 -> SparkFun-Passives:RESISTORKIT
Other:
- moved on the sheet: R1
Changed lines of the file:
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@@
 </variantdefs>
 <classes>
-<class number="0" name="default" width="0" drill="0">
+<class number="0" name="default" width="0.254" drill="0">
+<clearance class="0" value="0.1778"/>
 </class>
 </classes>
 <parts>
 <part name="FRAME1" library="frames" library_urn="urn:adsk.eagle:library:229" deviceset="A4L-LOC" device=""/>
-<part name="R1" library="SparkFun-Passives" deviceset="RESISTOR" device="AXIAL-0.3"/>
 <part name="D1" library="modified-sparkfun-parts" deviceset="LED" device="5MM"/>
 <part name="S1" library="modified-sparkfun-parts" deviceset="SWITCH" device="MAIN"/>
 <part name="H1" library="modified-sparkfun-parts" deviceset="COIN_CELL_HOLDER" device=""/>
+<part name="R1" library="SparkFun-Passives" deviceset="RESISTOR" device="KIT" value="100"/>
 </parts>
 <sheets>
@@
 <instances>
 <instance part="FRAME1" gate="G$1" x="0" y="0"/>
-<instance part="R1" gate="G$1" x="111.76" y="139.7" rot="R90"/>
 <instance part="D1" gate="G$1" x="111.76" y="129.54"/>
 <instance part="S1" gate="G$1" x="104.14" y="154.94"/>
 <instance part="H1" gate="G$1" x="93.98" y="129.54" rot="R270"/>
+<instance part="R1" gate="G$1" x="111.76" y="142.24" rot="R90"/>
 </instances>
 <busses>
@@
 </segment>
 </net>
-<net name="N$3" class="0">
-<segment>
-<pinref part="R1" gate="G$1" pin="1"/>
-<pinref part="D1" gate="G$1" pin="A"/>
-<wire x1="111.76" y1="134.62" x2="111.76" y2="132.08" width="0.1524" layer="91"/>
-</segment>
-</net>
-<net name="N$12" class="0">
-<segment>
-<pinref part="R1" gate="G$1" pin="2"/>
-<wire x1="111.76" y1="149.86" x2="111.76" y2="147.32" width="0.1524" layer="91"/>
-<pinref part="S1" gate="G$1" pin="1"/>
-<wire x1="111.76" y1="147.32" x2="111.76" y2="144.78" width="0.1524" layer="91"/>
-<wire x1="108.712" y1="157.48" x2="111.76" y2="157.48" width="0.1524" layer="91"/>
-<wire x1="111.76" y1="157.48" x2="111.76" y2="149.86" width="0.1524" layer="91"/>
-</segment>
-</net>
 <net name="N$1" class="0">
 <segment>
@@
 </segment>
 </net>
+<net name="N$3" class="0">
+<segment>
+<pinref part="S1" gate="G$1" pin="1"/>
+<wire x1="108.712" y1="157.48" x2="111.76" y2="157.48" width="0.1524" layer="91"/>
+<pinref part="R1" gate="G$1" pin="2"/>
+<wire x1="111.76" y1="157.48" x2="111.76" y2="147.32" width="0.1524" layer="91"/>
+</segment>
+</net>
+<net name="N$4" class="0">
+<segment>
+<pinref part="R1" gate="G$1" pin="1"/>
+<pinref part="D1" gate="G$1" pin="A"/>
+<wire x1="111.76" y1="137.16" x2="111.76" y2="132.08" width="0.1524" layer="91"/>
+</segment>
+</net>
